File: Chergo.kicad_pcb (KiCad board)
At the start: 2 copper layers, 124 x 102 mm, 20 parts, among them K1 KEYSW, K10 KEYSW, K11 KEYSW, K12 KEYSW, K13 KEYSW, K14 KEYSW, K15 KEYSW, K16 KEYSW, K17 KEYSW, K2 KEYSW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

Commit message: added silkscreen
Parts:
- added G***: LOGO, imagefootprints:BudgyHeadright, F.Cu at (160.4, 122.0)
- added G***: LOGO, imagefootprints:BudgyHeadleft, B.Cu at (160.4, 122.0)
- added G***: LOGO, imagefootprints:qmk25mm, B.Cu at (106.8, 70.2)
- moved G*** 47.3 mm to (106.5, 70.1)
